File: Hardware/PCB/Printrhub_Rev_0.3.brd (EAGLE design)
At the start: 82.5 x 61.2 mm, 69 parts, among them J1 DM3D-SF, SW1 SPST_TACT-KMR2, SW2 SPST_TACT-KMR2, U1 MK20DX256VLH7, U2 AP1117E, U3 MAX308-SOT23, Y2 16Mhz/8pF

Commit message: Updated to latest version of 0.3. This is the one that went to the board house.
Parts:
- removed EXP2: (no value), appfruits:1X06_SMD_STRAIGHT_ALT
- added JP2: (no value), pinhead+:2X05_SMT
- added R8: 1K, appfruits:0603-RES
- JP3: value M022.54MM_SCREWTERM -> M024UCON-15767; device SparkFun-Connectors:1X02_2.54_SCREWTERM -> SparkFun-Connectors:JST-2-SMD-VERT
- moved R4 10.5 mm to (2.29, 7.08)
- moved R13 6.35 mm to (2.29, 8.73), turned to 180 degrees
- moved U$38 6.10 mm to (7.62, 2.54)
- moved R19 5.08 mm to (47.0, 2.29)
- moved R16 5.08 mm to (54.6, 2.29)
- moved R17 5.08 mm to (52.1, 2.29)
- moved R18 5.08 mm to (49.5, 2.29)
- moved C1 4.78 mm to (26.0, 12.2), turned to 270 degrees
- moved JP3 3.24 mm to (49.5, 57.2)
- moved J1 3.18 mm to (34.3, 4.67)
- moved R23 3.17 mm to (41.9, 16.1)
- moved R27 3.17 mm to (41.9, 8.73)
- moved U$39 3.05 mm to (4.83, 55.8)
- moved C2 0.40 mm to (31.8, 32.1)
- moved D4 0.13 mm to (27.8, 59.8)
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Connections:
- removed net ESP_GPIO12: EXP2.2, X1.6
- new net RX2: JP2.9, U1.2
- new net SCL1: JP2.3, U1.55
- new net SDA1: JP2.5, U1.56
- new net TX2: JP2.7, U1.1
- net 3.3V: now also JP2.1
- net ESP_GPIO16: now also JP2.4; no longer EXP2.3
- net ESP_GPIO5: now also U1.27; no longer U1.1
- net EXT_VIN: now also JP3.VCC; no longer JP3.P2
- net GND: now also JP2.2, JP3.GND, R8.1; no longer EXP2.6, JP3.P1
- net LCD_RESET: now also U1.45; no longer U1.55
- net MK20_GPIO_14: now also JP2.6, X1.6; no longer EXP2.5
- net MK20_GPIO_2: now also JP2.8; no longer EXP2.4
- net RESET_B: now also JP2.10, R8.2; no longer EXP2.1
Routing:
- net TX2: track 0.00 -> 56.0 mm, vias 0 -> 2
- net RX2: track 0.00 -> 55.6 mm, vias 0 -> 2
- net SCL1: track 0.00 -> 48.8 mm, vias 0 -> 2
- net SDA1: track 0.00 -> 48.5 mm, vias 0 -> 2
- net RESET_B: track 53.6 -> 73.7 mm
- net N$10: track 2.92 -> 16.6 mm, vias 0 -> 2
- net ESP_GPIO5: track 32.2 -> 21.0 mm, vias 2 -> 0
- net MK20_GPIO_14: track 50.8 -> 40.9 mm
- net ESP_RESET: track 169.7 -> 179.3 mm
- net N$5: track 2.86 -> 12.1 mm
- net ESP_GPIO12: track 7.59 -> 0.00 mm
- net ESP_GPIO16: track 10.0 -> 3.76 mm
- net 3.3V: track 75.5 -> 78.4 mm, vias 36 -> 37
- net LCD_LITE: track 17.9 -> 20.6 mm
- net MK20_GPIO_3: track 53.2 -> 55.6 mm
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Other:
- board text added: "DNI"
- board text added: "EXP"
- board text removed: "E12"
- board text removed: "E16"
- board text removed: "GND"
- board text removed: "M02"
- board text removed: "M14"
- board text removed: "RES_B"
