File: Hardware/PCB/Printrhub_Rev_0.3.sch (EAGLE design)
At the start: 69 parts, among them J1 DM3D-SF, SW1 SPST_TACT-KMR2, SW2 SPST_TACT-KMR2, U1 MK20DX256VLH7, U2 AP1117E, U3 MAX308-SOT23, Y2 16Mhz/8pF

Commit message: Updated to latest version of 0.3. This is the one that went to the board house.
Parts:
- removed EXP2: (no value), appfruits:M06SMD-STRAIGHT-ALT
- added JP2: (no value), pinhead+:PINHD-2X5SMT
- added R8: 1K, appfruits:RESISTOR-1K
- JP3: value M022.54MM_SCREWTERM -> M024UCON-15767; device SparkFun-Connectors:M022.54MM_SCREWTERM -> SparkFun-Connectors:M024UCON-15767
Connections:
- removed net ESP_GPIO12: EXP2.2, X1.GPIO12
- new net RX2: JP2.9, U1.PTE1
- new net SCL1: JP2.3, U1.PTC10
- new net SDA1: JP2.5, U1.PTC11
- new net TX2: JP2.7, U1.PTE0
- net 3.3V: now also JP2.1
- net ESP_GPIO16: now also JP2.4; no longer EXP2.3
- net ESP_GPIO5: now also U1.PTA5; no longer U1.PTE0
- net GND: now also JP2.2, R8.1; no longer EXP2.6
- net LCD_RESET: now also U1.PTC2; no longer U1.PTC10
- net MK20_GPIO_14: now also JP2.6, X1.GPIO12; no longer EXP2.5
- net MK20_GPIO_2: now also JP2.8; no longer EXP2.4
- net RESET_B: now also JP2.10, R8.2; no longer EXP2.1
Other:
- note added: "Do not install"
- note removed: "USB-Connector"
- moved on the sheet: JP3
